File: KiCad/atmega32u4_17keynumpad.kicad_sch (KiCad schematic)
At the start: 39 parts, among them J1 Conn_01x03_Pin, J2 power connector, J3 LCD1602, SW1 SW_Push, SW1 slide_switch, SW10 SW_Push, SW11 SW_Push, SW12 SW_Push, SW13 SW_Push, SW14 SW_Push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

Commit message: pcb fix
Parts:
- removed J2: power connector, Connector_PinHeader_2.54mm:PinHeader_1x02_P2.54mm_Vertical, symbol Altium Content Vault:root_0_3bc925449376181038e59eaffc5286c_Altium Content Vault
- removed J3: LCD1602, Connector_PinHeader_2.54mm:PinHeader_1x04_P2.54mm_Vertical, symbol Altium Content Vault:root_2_Header_Male_1R_04P_Altium Content Vault
- removed SW1: slide_switch, Button_Switch_THT:SW_Slide-03_Wuerth-WS-SLTV_10x2.5x6.4_P2.54mm, symbol Altium Content Vault:root_0_ec4e4964ed0d2d669af15d5af94fda9_Altium Content Vault
- added J3: power supply, Connector_PinSocket_2.54mm:PinSocket_1x02_P2.54mm_Vertical, symbol Connector:Conn_01x02_Pin
- added J4: LCD1602, Connector_PinHeader_2.54mm:PinHeader_1x04_P2.54mm_Vertical, symbol Connector:Conn_01x04_Pin
- added SW19: slide switch, Button_Switch_THT:SW_Slide-03_Wuerth-WS-SLTV_10x2.5x6.4_P2.54mm, symbol Switch:SW_SPDT
Connections:
- net +3V8: now also J4.3 (Pin_3), SW19.3 (C)
- net GND: now also J3.1 (Pin_1), J4.4 (Pin_4)
- net Pin 8 (ROW 1): now also D1.1 (K)
- net SCL: now also J4.1 (Pin_1)
- net SDA: now also J4.2 (Pin_2)
- net at SW1.1: now also D1.2 (A)
- new net: J3.2 (Pin_2), SW19.2 (B)
- no-connect marks 7 -> 8
Other:
- moved on the sheet: SW1, SW2, SW3, SW4

Commit message: finished pcb
Parts:
- removed SW19: slide switch, Button_Switch_THT:SW_Slide-03_Wuerth-WS-SLTV_10x2.5x6.4_P2.54mm, symbol Switch:SW_SPDT
- added SW18: slide_switch, Button_Switch_THT:SW_Slide-03_Wuerth-WS-SLTV_10x2.5x6.4_P2.54mm, symbol Switch:SW_SPDT_XKB_DMx-xxxx-1
- SW11, SW15, SW17: footprint PCM_Switch_Keyboard_Cherry_MX:SW_Cherry_MX_PCB_1.00u -> PCM_Switch_Keyboard_Cherry_MX:SW_Cherry_MX_PCB_2.00u
- renumbered J3 to J2, J4 to J3
Connections:
- net +3V8: now also J3.2 (Pin_2), SW18.2 (B); no longer J3.3 (Pin_3)
- net GND: now also J3.1 (Pin_1); no longer J3.4 (Pin_4)
- net Pin 10 (COL 4): now also SW11.1, SW17.1, SW4.1; no longer SW11.2, SW17.2, SW4.2
- net Pin 14 (COL 2): now also SW13.1, SW15.1, SW2.1, SW6.1, SW9.1; no longer SW13.2, SW15.2, SW2.2, SW6.2, SW9.2
- net Pin 16 (COL 3): now also SW10.1, SW14.1, SW16.1, SW3.1, SW7.1; no longer SW10.2, SW14.2, SW16.2, SW3.2, SW7.2
- net Pin 9 (COL 1): now also SW1.1, SW12.1, SW5.1, SW8.1; no longer SW1.2, SW12.2, SW5.2, SW8.2
- net SCL: now also J3.4 (Pin_4); no longer J3.1 (Pin_1)
- net SDA: now also J3.3 (Pin_3); no longer J3.2 (Pin_2)
- net at D5.2 (A): now also SW5.2; no longer SW5.1
- net at D6.2 (A): now also SW6.2; no longer SW6.1
- net at D14.2 (A): now also SW14.2; no longer SW14.1
- net at D8.2 (A): now also SW8.2; no longer SW8.1
- net at D2.2 (A): now also SW2.2; no longer SW2.1
- net at D3.2 (A): now also SW3.2; no longer SW3.1
- net at D17.2 (A): now also SW17.2; no longer SW17.1
- net at D13.2 (A): now also SW13.2; no longer SW13.1
- net at D7.2 (A): now also SW7.2; no longer SW7.1
- net at D10.2 (A): now also SW10.2; no longer SW10.1
- net at J2.2 (Pin_2): now also SW18.1 (A)
- net at D11.2 (A): now also SW11.2; no longer SW11.1
- net at D16.2 (A): now also SW16.2; no longer SW16.1
- net at D15.2 (A): now also SW15.2; no longer SW15.1
- net at D4.2 (A): now also SW4.2; no longer SW4.1
- net at D1.2 (A): now also SW1.2; no longer SW1.1
- net at D9.2 (A): now also SW9.2; no longer SW9.1
- net at D12.2 (A): now also SW12.2; no longer SW12.1
Other:
- moved on the sheet: J2, J3, SW1, SW10, SW11, SW12, SW13, SW14, SW15, SW16, SW17, SW2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
